Commit message: Add sensors

File: catkin_ws/src/my_robot/urdf/my_robot.xacro (robot description, xacro)
@@ -117,3 +117,79 @@
     <dynamics damping="1.0" friction="1.0"/>
   </joint>
+<link name='camera'>
+ <pose>0 0 0 0 0 0</pose>
+      <inertial>
+      <mass value="0.1"/>
+      <origin xyz="0.05 0.05 0.05" rpy="0 0 0"/>
+      <inertia
+          ixx="1e-6" ixy="0" ixz="0"
+          iyy="1e-6" iyz="0"
+          izz="1e-6"
+      />
+    </inertial>
+    <collision>
+      <origin xyz="0 0 0" rpy="0 0 0"/>
+      <geometry>
+        <box size=".05 .05 .05" />
+      </geometry>
+    </collision>
+    <visual>
+      <origin xyz="0 0 0" rpy="0 0 0"/>
+     <geometry>
+         <box size=".05 .05 .05" />
+      </geometry>
+    </visual>
+  </link>
+<joint type="fixed" name="camera_joint">
+    <origin xyz="0.2 0 0" rpy="0 0 0"/>
+    <child link="camera"/>
+    <parent link="chassis"/>
+    <axis xyz="0 1 0" rpy="0 0 0"/>
+  </joint>
+<link name='hokuyo'>
+ <pose>0 0 0 0 0 0</pose>
+      <inertial>
+      <mass value="1e-5"/>
+      <origin xyz="0 0 0" rpy="0 0 0"/>
+      <inertia
+          ixx="1e-6" ixy="0" ixz="0"
+          iyy="1e-6" iyz="0"
+          izz="1e-6"
+      />
+    </inertial>
+    <collision>
+      <origin xyz="0 0 0" rpy="0 0 0"/>
+      <geometry>
+        <box size=".1 .1 .1" />
+      </geometry>
+    </collision>
+    <visual>
+      <origin xyz="0 0 0" rpy="0 0 0"/>
+     <geometry>
+       <mesh filename="package://my_robot/meshes/hokuyo.dae">
+       </mesh>
+      </geometry>
+    </visual>
+  </link>
+<joint type="fixed" name="hokuyo_joint">
+    <origin xyz="0.15 0 0.1" rpy="0 0 0"/>
+    <child link="hokuyo"/>
+    <parent link="chassis"/>
+    <axis xyz="0 1 0" rpy="0 0 0"/>
+  </joint>
+<gazebo reference="left_wheel">
+    <material>Gazebo/Black</material>
+</gazebo>
+<gazebo reference="right_wheel">
+    <material>Gazebo/Black</material>
+</gazebo>
+<gazebo reference="chassis">
+    <material>Gazebo/Gold</material>
+</gazebo>
+<gazebo reference="camera">
+    <material>Gazebo/Red</material>
+</gazebo>
+<gazebo reference="hokuyo">
+    <material>Gazebo/Green</material>
+</gazebo>
 </robot>

Commit message: -finish project

File: catkin_ws/src/my_robot/urdf/my_robot.xacro (robot description, xacro)
@@ -9,5 +9,5 @@
   </joint>
   <link name='chassis'>
-    <pose>0 0 0.1 0 0 0</pose>
+    <pose>0 0 0.2 0 0 0</pose>
     <inertial>
       <mass value="15.0"/>
@@ -22,5 +22,5 @@
       <origin xyz="0 0 0" rpy=" 0 0 0"/>
       <geometry>
-        <box size=".4 .2 .1"/>
+        <box size=".4 .3 .2"/>
       </geometry>
     </collision>
@@ -28,29 +28,53 @@
       <origin xyz="0 0 0" rpy=" 0 0 0"/>
       <geometry>
-        <box size=".4 .2 .1"/>
+        <box size=".4 .3 .2"/>
       </geometry>
     </visual>
     <collision name='back_caster_collision'>
-      <origin xyz="-0.15 0 -0.05" rpy=" 0 0 0"/>
-      <geometry>
-        <sphere radius="0.0499"/>
+      <origin xyz="-0.15 0 -0.175" rpy=" 0 0 0"/>
+      <geometry>
+        <sphere radius="0.0249"/>
       </geometry>
     </collision>
     <visual name='back_caster_visual'>
-      <origin xyz="-0.15 0 -0.05" rpy=" 0 0 0"/>
-      <geometry>
-        <sphere radius="0.05"/>
+      <origin xyz="-0.15 0 -0.175" rpy=" 0 0 0"/>
+      <geometry>
+        <sphere radius="0.025"/>
+      </geometry>
+    </visual>
+     <collision name='back_caster_collision_base'>
+      <origin xyz="-0.15 0 -0.125" rpy=" 0 0 0"/>
+      <geometry>
+         <cylinder radius="0.025" length="0.1"/>
+      </geometry>
+    </collision>
+    <visual name='back_caster_visual_base'>
+      <origin xyz="-0.15 0 -0.125" rpy=" 0 0 0"/>
+      <geometry>
+         <cylinder radius="0.025" length="0.1"/>
       </geometry>
     </visual>
     <collision name='front_caster_collision'>
-      <origin xyz="0.15 0 -0.05" rpy=" 0 0 0"/>
-      <geometry>
-        <sphere radius="0.0499"/>
+      <origin xyz="0.15 0 -0.175" rpy=" 0 0 0"/>
+      <geometry>
+        <sphere radius="0.0249"/>
       </geometry>
     </collision>
     <visual name='front_caster_visual'>
-      <origin xyz="0.15 0 -0.05" rpy=" 0 0 0"/>
-      <geometry>
-        <sphere radius="0.05"/>
+      <origin xyz="0.15 0 -0.175" rpy=" 0 0 0"/>
+      <geometry>
+        <sphere radius="0.025"/>
+      </geometry>
+    </visual>
+     <collision name='front_caster_collision_base'>
+      <origin xyz="0.15 0 -0.125" rpy=" 0 0 0"/>
+      <geometry>
+         <cylinder radius="0.025" length="0.1"/>
+      </geometry>
+    </collision>
+    <visual name='front_caster_visual_base'>
+      <origin xyz="0.15 0 -0.125" rpy=" 0 0 0"/>
+      <geometry>
+         <cylinder radius="0.025" length="0.1"/>
       </geometry>
     </visual>
@@ -69,5 +93,5 @@
       <origin xyz="0 0 0" rpy="0 1.5707 1.5707"/>
       <geometry>
-        <cylinder radius="0.1" length="0.05"/>
+        <cylinder radius="0.2" length="0.05"/>
       </geometry>
     </collision>
@@ -75,5 +99,5 @@
       <origin xyz="0 0 0" rpy="0 1.5707 1.5707"/>
      <geometry>
-        <cylinder radius="0.1" length="0.05"/>
+        <cylinder radius="0.2" length="0.05"/>
       </geometry>
     </visual>
@@ -92,5 +116,5 @@
       <origin xyz="0 0 0" rpy="0 1.5707 1.5707"/>
       <geometry>
-        <cylinder radius="0.1" length="0.05"/>
+        <cylinder radius="0.2" length="0.05"/>
       </geometry>
     </collision>
@@ -98,10 +122,10 @@
       <origin xyz="0 0 0" rpy="0 1.5707 1.5707"/>
      <geometry>
-        <cylinder radius="0.1" length="0.05"/>
+        <cylinder radius="0.2" length="0.05"/>
       </geometry>
     </visual>
   </link>
  <joint type="continuous" name="left_wheel_hinge">
-    <origin xyz="0 0.15 0" rpy="0 0 0"/>
+    <origin xyz="0 0.20 0" rpy="0 0 0"/>
     <child link="left_wheel"/>
     <parent link="chassis"/>
@@ -111,5 +135,5 @@
   </joint>
 <joint type="continuous" name="right_wheel_hinge">
-    <origin xyz="0 -0.15 0" rpy="0 0 0"/>
+    <origin xyz="0 -0.20 0" rpy="0 0 0"/>
     <child link="right_wheel"/>
     <parent link="chassis"/>
@@ -148,6 +172,6 @@
     <axis xyz="0 1 0" rpy="0 0 0"/>
   </joint>
-<link name='hokuyo'>
- <pose>0 0 0 0 0 0</pose>
+<link name='hokuyo_base'>
+  <pose>0 0 0 0 0 0</pose>
       <inertial>
       <mass value="1e-5"/>
@@ -162,4 +186,34 @@
       <origin xyz="0 0 0" rpy="0 0 0"/>
       <geometry>
+        <box size="0.05 0.05 0.2" />
+      </geometry>
+    </collision>
+    <visual>
+      <origin xyz="0 0 0" rpy="0 0 0"/>
+     <geometry>
+         <box size="0.05 0.05 .2" />
+      </geometry>
+    </visual>
+  </link>
+<joint type="fixed" name="hokuyo_base_joint">
+    <origin xyz="0.15 0 0.2" rpy="0 0 0"/>
+    <child link="hokuyo_base"/>
+    <parent link="chassis"/>
+    <axis xyz="0 1 0" rpy="0 0 0"/>
+  </joint>
+<link name='hokuyo'>
+ <pose>0 0 0 0 0 0</pose>
+      <inertial>
+      <mass value="1e-5"/>
+      <origin xyz="0 0 0" rpy="0 0 0"/>
+      <inertia
+          ixx="1e-6" ixy="0" ixz="0"
+          iyy="1e-6" iyz="0"
+          izz="1e-6"
+      />
+    </inertial>
+    <collision>
+      <origin xyz="0 0 0" rpy="0 0 0"/>
+      <geometry>
         <box size=".1 .1 .1" />
       </geometry>
@@ -174,5 +228,5 @@
   </link>
 <joint type="fixed" name="hokuyo_joint">
-    <origin xyz="0.15 0 0.1" rpy="0 0 0"/>
+    <origin xyz="0.15 0 0.3" rpy="0 0 0"/>
     <child link="hokuyo"/>
     <parent link="chassis"/>
@@ -194,3 +248,6 @@
     <material>Gazebo/Green</material>
 </gazebo>
+<gazebo reference="hokuyo_base">
+    <material>Gazebo/Green</material>
+</gazebo>
 </robot>
