Commit message: finish project

File: amcl/catkin_ws/src/my_robot2/urdf/my_robot.xacro (robot description, xacro)
@@ -186,5 +186,5 @@
       <origin xyz="0 0 0" rpy="0 0 0"/>
       <geometry>
-        <box size="0.05 0.05 0.2" />
+        <box size="0.05 0.05 0.1" />
       </geometry>
     </collision>
@@ -192,10 +192,10 @@
       <origin xyz="0 0 0" rpy="0 0 0"/>
      <geometry>
-         <box size="0.05 0.05 .2" />
+         <box size="0.05 0.05 .1" />
       </geometry>
     </visual>
   </link>
 <joint type="fixed" name="hokuyo_base_joint">
-    <origin xyz="0.15 0 0.2" rpy="0 0 0"/>
+    <origin xyz="0.15 0 0.15" rpy="0 0 0"/>
     <child link="hokuyo_base"/>
     <parent link="chassis"/>
@@ -228,5 +228,5 @@
   </link>
 <joint type="fixed" name="hokuyo_joint">
-    <origin xyz="0.15 0 0.3" rpy="0 0 0"/>
+    <origin xyz="0.15 0 0.2" rpy="0 0 0"/>
     <child link="hokuyo"/>
     <parent link="chassis"/>
