Commit message: finsih project

File: map/catkin_ws/src/my_robot3/urdf/my_robot.xacro (robot description, xacro)
@@ -36,4 +36,14 @@
         <sphere radius="0.0249"/>
       </geometry>
+        <surface>
+        <friction>
+          <ode>
+            <mu>0</mu>
+            <mu2>0</mu2>
+            <slip1>1.0</slip1>
+            <slip2>1.0</slip2>
+          </ode>
+        </friction>
+      </surface>
     </collision>
     <visual name='back_caster_visual'>
@@ -60,4 +70,14 @@
         <sphere radius="0.0249"/>
       </geometry>
+        <surface>
+        <friction>
+          <ode>
+            <mu>0</mu>
+            <mu2>0</mu2>
+            <slip1>1.0</slip1>
+            <slip2>1.0</slip2>
+          </ode>
+        </friction>
+      </surface>
     </collision>
     <visual name='front_caster_visual'>
@@ -145,5 +165,5 @@
  <pose>0 0 0 0 0 0</pose>
       <inertial>
-      <mass value="0.1"/>
+      <mass value="0"/>
       <origin xyz="0.05 0.05 0.05" rpy="0 0 0"/>
       <inertia
@@ -174,5 +194,5 @@
  <joint name="camera_optical_joint" type="fixed">
     <origin xyz="0 0 0" rpy="-1.5707 0 -1.5707"/>
-    <parent link="camera_link"/>
+    <parent link="camera"/>
     <child link="camera_link_optical"/>
   </joint>
@@ -182,5 +202,5 @@
   <pose>0 0 0 0 0 0</pose>
       <inertial>
-      <mass value="1e-5"/>
+      <mass value="0"/>
       <origin xyz="0 0 0" rpy="0 0 0"/>
       <inertia

Commit message: Finish project

File: map/catkin_ws/src/my_robot3/urdf/my_robot.xacro (robot description, xacro)
@@ -34,5 +34,5 @@
       <origin xyz="-0.15 0 -0.175" rpy=" 0 0 0"/>
       <geometry>
-        <sphere radius="0.0249"/>
+        <sphere radius="0.0248"/>
       </geometry>
         <surface>
@@ -68,5 +68,5 @@
       <origin xyz="0.15 0 -0.175" rpy=" 0 0 0"/>
       <geometry>
-        <sphere radius="0.0249"/>
+        <sphere radius="0.0248"/>
       </geometry>
         <surface>
